File: RP2040-Shim-2.brd (EAGLE design)
At the start: 46 x 22.9 mm, 43 parts, among them SW1 KMR2, U1 RP2040_QFN56, U2 2MB Flash, U3 AP2112-3.3, U4 PMS150C-6PIN, Y1 12MHZ

Commit message: Update osc caps to 15 pF, add pinout diagram
Parts:
- C10, C11: value 12pF -> 15pF
Changed lines of the file:
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@@
 <attribute name="VALUE" x="27.235" y="21.305" size="1.27" layer="27" rot="R180"/>
 </element>
-<element name="C11" library="rcl" package="C0402K" value="12pF" x="35.9" y="3.5" smashed="yes">
+<element name="C11" library="rcl" package="C0402K" value="15pF" x="35.9" y="3.5" smashed="yes">
 <attribute name="NAME" x="34.5" y="2.18" size="0.8128" layer="25" font="vector" ratio="15"/>
 <attribute name="VALUE" x="35.4" y="2.05" size="1.016" layer="27"/>
 </element>
-<element name="C10" library="rcl" package="C0402K" value="12pF" x="35.9" y="8.3" smashed="yes">
+<element name="C10" library="rcl" package="C0402K" value="15pF" x="35.9" y="8.3" smashed="yes">
 <attribute name="NAME" x="34.675" y="7.5" size="0.6096" layer="25" font="vector" ratio="15" rot="R90"/>
 <attribute name="VALUE" x="35.4" y="6.85" size="1.016" layer="27"/>
